File: nixieclock/nixieclock.kicad_sch (KiCad schematic)
At the start: 0 parts

Commit message: finalized design ready for quality check
Parts:
- added H1, H2, H3, H4: MountingHole, MountingHole:MountingHole_5.3mm_M5_Pad, symbol Mechanical:MountingHole
