File: nixieclock.kicad_pcb (KiCad board)
At the start: 4 copper layers, 120 x 93 mm, 186 parts, among them J1 USB_C_Receptacle_USB2.0, J2 Conn_ARM_JTAG_SWD_10, Q10 BSS131, Q11 BSS131, Q12 BSS131, Q13 BSS131, Q14 BSS131, Q15 BSS131, Q16 BSS131, Q17 BSS131, Q18 BSS131, Q19 BSS131, Q2 IRLR3110ZTRPBF, Q20 BSS131, Q21 BSS131, Q22 BSS131, Q23 BSS131, Q24 BSS131, Q25 BSS131, Q26 BSS131, Q27 BSS131, Q28 BSS131, Q29 BSS131, Q3 BSR92P, Q30 BSS131, Q31 BSS131, Q32 BSS131, Q33 BSS131, Q34 BSS131, Q35 BSS131, Q36 BSS131, Q37 BSS131, Q38 BSS131, Q39 BSS131, Q4 BSR92P, Q40 BSS131, Q41 BSS131, Q42 BSS131, Q43 BSS131, Q44 BSS131, Q45 BSS131, Q46 BSS131, Q47 BSS131, Q48 BSS131, Q5 BSS131, Q6 BSS131, Q7 BSS131, Q8 BSS131, Q9 BSS131, SW1 EN11-VSM, U1 LT3757AEMSE, U2 AMS1117-3.3, U3 74HC595, U4 74HC595, U5 74HC595, U6 74HC595, U7 74HC595, U8 STM32F051R4Tx, Y1 8MHz, Y2 32.768kHz

Commit message: finalized design; fixed NE-2 bulb work
Parts:
- moved R26 1.70 mm to (110.8, 120.8), turned to -90 degrees
- moved R25 1.15 mm to (108.4, 120.8)
Connections:
- J1 pad A5: unconnected-(J1-PadA5) -> (no net)
- J1 pad A6: unconnected-(J1-PadA6) -> (no net)
- J1 pad A7: unconnected-(J1-PadA7) -> (no net)
- J1 pad A8: unconnected-(J1-PadA8) -> (no net)
- J1 pad B5: unconnected-(J1-PadB5) -> (no net)
- J1 pad B6: unconnected-(J1-PadB6) -> (no net)
- J1 pad B7: unconnected-(J1-PadB7) -> (no net)
- J1 pad B8: unconnected-(J1-PadB8) -> (no net)
- NE1 pad 1: Net-(NE1-Pad1) -> /nixie_tubes/NEH-
- NE2 pad 1: Net-(NE1-Pad1) -> /nixie_tubes/NEH-
- NE2 pad 2: Net-(NE1-Pad2) -> Net-(NE2-Pad2)
- Q3 pad 2: /nixie_tubes/NEH+ -> HV
- Q3 pad 3: HV -> /nixie_tubes/NEH+
- Q4 pad 2: /nixie_tubes/NEH- -> HV
- Q4 pad 3: HV -> /nixie_tubes/NEH-
- R26 pad 1: Net-(NE1-Pad1) -> /nixie_tubes/NEH+
- R26 pad 2: /nixie_tubes/NEH- -> Net-(NE2-Pad2)
Routing:
- net Net-(NE2-Pad2): track 0.00 -> 10.3 mm
- net HV: track 102.1 -> 112.2 mm
- net /nixie_tubes/NEH-: track 36.3 -> 44.4 mm
- net Net-(NE1-Pad1): track 7.94 -> 0.00 mm
- net /nixie_tubes/NEH+: track 23.8 -> 30.2 mm
- net /cathode_registers/GC1: track 66.7 -> 61.9 mm
- net Net-(NE1-Pad2): track 8.01 -> 3.27 mm
- net /cathode_registers/GC2: track 71.4 -> 66.7 mm
- net /cathode_registers/GC9: track 46.7 -> 45.3 mm
Other:
- rule pad_to_mask_clearance: 0 -> 0.05
- board text removed: "Made with love for Clair, Happy Birthday"
